File: hardware/kicad/01-alimentacion.kicad_sch (KiCad schematic)
At the start: 37 parts, among them J1 PSU 5V 5A, Q1 AO3401, Q2 2N7000, Q3 AO3401, Q4 2N7000, Q5 2N7000, SW1 RESET gabinete, U1 XY-SJVA 6.85V/0.6A, U2 XL6019, U3 CD4541BE, U4 NE555P

Commit message: Lock v1 proto hardware: 5 V MOSFET OR, THT parts, 2 IN / 2 OUT, independent buzzer.
PCF keeps NET and ALARM LEDs; buzzer is P3 via ULN so a rule can sound without closing field relays.

Co-authored-by: Cursor <cursoragent@cursor.com>
Parts:
- removed C2: 1000uF/16V, symbol Device:C_Polarized
- removed D1: SB560, symbol Device:D_Schottky
- removed Q2, Q4: 2N7000, symbol Transistor_FET:2N7000
- added C10, C17, C8, C9: 100n, symbol Device:C
- added J7: IDC A→B, symbol Module:IDC10
- added Q10, Q8: NDP6020P, symbol Device:Q_PMOS
- added Q11, Q9: 2N7000, symbol Transistor_FET:2N7000
- added R18, R20, R24, R36, R37: 100k, symbol Device:R
- added R19, R23: 1k, symbol Device:R
- added U13: 74HCT125, symbol Module:AHCTBUF
- Q1, Q3: value AO3401 -> NDP6020P
- U4: value NE555P -> TLC555
Connections:
- net 5V_MODEM: now also J7.4 (5V_MODEM); no longer Q3.G, R4.1
- net 5V_PSU: now also Q8.D
- net 5V_SYS: now also J7.2 (5V_SYS), J7.8 (LED_PWR)
- net BTN_RESET: now also J7.9 (BTN_RESET)
- net GEL_ADC: now also J7.5 (GEL_ADC)
- net GND: now also Q3.G, R4.1, C10.1, C10.2, C17.1, C17.2, C8.1, C8.2, C9.1, C9.2, J7.1 (GND), J7.10 (GND), J7.3 (GND), Q10.D, Q10.G, Q10.S, Q11.1 (S), Q11.3 (D), Q8.S, Q9.1 (S), R18.2, R20.2, R24.2, R36.2, R37.1, R37.2, U13.1 (1OE), U13.10 (3OE), U13.12 (4A), U13.13 (4OE), U13.14 (VCC), U13.3 (1Y), U13.4 (2A), U13.6 (2OE), U13.7 (GND), U13.9 (3A)
- net IO15: now also J7.6 (IO15)
- net MODEM_CUT: now also J7.7 (MODEM_CUT), R23.1
- net WDT_MR: now also R20.1
- net WDT_PULSE: now also R19.1
- net at Q1.G, R3.1: now also R19.2
- net PSU_DET: now reaches Q5.2 (G), R1.2
- net PSU_DET: now also Q9.2 (G), R18.1
- net BB_EN: now reaches Q5.3 (D), R2.2, U2.3 (EN)
- net BB_EN: now also Q11.2 (G)
- new net: R23.2, R24.1, U13.2 (1A)
- new net: Q8.G, Q9.3 (D), R36.1
Other:
- note added: "Ajuste XL6019 5,1 V (ya no 5,4: no hay Schottky). No XL6009 / ZK-4KX."
- note added: "Cinta 10: GND en 1/3/10. Polarizada. No enchufar con 5 V. 1000uF del modem va en B."
- note added: "D5: timeout 4541 baja TRIG. SW1 NA a GND. TLC555 OUT a Q1 (no NE555 bipolar)."
- note added: "Hay PSU: Q5/Q9 ON -> backup EN=0, Q8 ON, Q10 OFF."
- note added: "Patada IO15 acople. No DC a GND en IO15. R20 baja MR."
- note added: "Q1 5V_SYS. 555 idle LOW = ON. Pulso HIGH ~2 s = OFF."
- note added: "Q3 5V_MODEM. 74HCT125 DIP-14: 1=OE 2=A 3=Y 7=GND 14=VCC. 6/10/13→VCC, 4/9/12→GND."
- note added: "R8/C4: tunear 4-5 min (2^16). Pin 9 HIGH => Q activo bajo. C8 junto al 4541."
- note added: "Sin PSU: Q8 OFF, EN=Gel+, Q11 ON, Q10 ON. Ambos NDP6020P S=BUS D=fuente."
- note added: "TLC555 HIGH=5V corta Q1. Modem: 74HCT125 DIP (3V3 in, 5V out). Todo THT."
- note added: "WDT CD4541 (~4-5 min) + TLC555 CMOS (~2 s) en 5V_BUS"
- note removed: "5V_PSU -> Q5 ON -> EN=GND -> backup OFF. Sin PSU -> R2 sube EN a Gel+."
- note removed: "AO3401 S=5V_BUS. Gate a GND = ON. 2N7000 sube el gate = OFF."
- note removed: "Ajuste 5,4 V. D1 SB560. XL6019 buck-boost auto. No XL6009 (solo boost). No ZK-4KX."
- note removed: "D5: timeout 4541 baja TRIG. SW1 NA a GND. OUT 555 = WDT_PULSE."
- note removed: "Patada IO15 acople. No DC a GND en IO15."
- note removed: "Q1 corta 5V_SYS ~2 s. Default ON."
- note removed: "Q3 5V_MODEM. GPIO de salida (no IO39, no IO2). C2 junto al A7672."
- note removed: "R8/C4: tunear 4-5 min (2^16). Pin 9 HIGH => Q activo bajo."
- note removed: "Si el modulo no tiene EN: AO3401 corta Gel+ a VIN."
- note removed: "WDT CD4541 (~4-5 min) + NE555 (~2 s) en 5V_BUS"

Commit message: Stop tracking PDFs and generated KiCad dumps; set WiFi from the web over Ethernet.
Vendor manuals, schematic PDFs, SVG previews and ERC reports do not belong in git or agent context. Firmware prefers Ethernet and accepts set_wifi/clear_wifi from the device page.

Co-authored-by: Cursor <cursoragent@cursor.com>
Parts:
- removed J7: IDC A→B, symbol Module:IDC10
- removed Q10, Q8: NDP6020P, symbol Device:Q_PMOS
- removed Q11, Q5, Q9: 2N7000, symbol Transistor_FET:2N7000
- removed R36, R37: 100k, symbol Device:R
- removed U13: 74HCT125, symbol Module:AHCTBUF
- added D10: 1N4148, symbol Device:D
- added J7: Enlace 5V A, symbol Connector_Generic:Conn_01x04
- added J9: Enlace sig A, symbol Connector_Generic:Conn_01x06
- added U13: 74HCT14, symbol Module:HCT14
- added U14: LM66200, symbol Module:LM66200
Connections:
- net 5V_MODEM: now also J7.4 (Pin_4)
- net 5V_PSU: now also U14.1 (VIN1)
- net 5V_SYS: now also J7.2 (Pin_2); no longer D2.2 (A), R5.2
- net BB_EN: now also D10.1 (K)
- net BTN_RESET: now also J9.5 (Pin_5)
- net GEL_ADC: now also J9.1 (Pin_1)
- net GND: now also J7.1 (Pin_1), J7.3 (Pin_3), J9.6 (Pin_6), U13.11 (5A), U13.13 (6A), U13.7 (GND), U13.9 (4A), U14.3 (GND), U14.5 (EN); no longer BT1.1 (+), C1.1, C10.1, C17.1, C7.1, C8.1, C9.1, F1.2, Q1.S, Q3.G, Q3.S, R11.1, R11.2, R12.1, R2.1, R4.1, R6.1, R9.1, U2.1 (VIN+), U2.4 (VOUT+), U3.10 (MODE), U3.12 (A), U3.13 (B), U3.14 (V_{DD}), U3.9 (Q/~{Q}_SELECT), U4.4 (~{RST}), U4.6 (THRES), U4.7 (DISCH), U4.8 (VCC)
- net IO15: now also J9.2 (Pin_2)
- net MODEM_CUT: now also J9.3 (Pin_3)
- net PSU_DET: now also D10.2 (A), U13.1 (1A), U13.2 (1Y)
- net at R23.2, R24.1: now also U13.3 (2A)
- new net: Q3.G, R4.1, U13.6 (3Y)
- new net: U14.2 (VIN2), U2.4 (VOUT+)
- new net 5V_BUS: C1.1, C10.1, C17.1, C7.1, C8.1, C9.1, Q1.S, Q3.S, R11.1, R11.2, R12.1, R9.1, U13.14 (VCC), U14.4 (VOUT), U3.10 (MODE), U3.12 (A), U3.13 (B), U3.14 (V_{DD}), U3.9 (Q/~{Q}_SELECT), U4.4 (~{RST}), U4.6 (THRES), U4.7 (DISCH), U4.8 (VCC)
- new net GEL_P: BT1.1 (+), F1.2, R2.1, R6.1, U2.1 (VIN+)
- new net LED_PWR: D2.2 (A), J9.4 (Pin_4), R5.2
- new net MC_BUF: U13.4 (2Y), U13.5 (3A)
- no-connect marks 2 -> 6
Other:
- note added: "Ajuste XL6019 5,1 V. No XL6009 / ZK-4KX. Modulo AE con pines 2,54."
- note added: "No cinta IDC. No 5V_BUS / 3V3 / GEL+. Luego una placa: estas nets son pistas."
- note added: "OR: LM66200 (VIN1=PSU, VIN2=XL6019). EN=0 con PSU (HCT14+D10). R2 a Gel+."
- note added: "Proto A↔B: J7 bornera 5,08 (GND 5V_SYS GND 5V_MODEM) + J9 Molex KK 2,54 o bornera."
- note added: "Q3 5V_MODEM. HCT14: 2Y->3A = buffer. D10: 1Y baja BB_EN (R2 a Gel+)."
- note added: "TLC555->Q1. 74HCT14: 1=EN backup, 2+3=buffer MODEM_CUT. Solo 2x NDP6020P."
- note removed: "Ajuste XL6019 5,1 V (ya no 5,4: no hay Schottky). No XL6009 / ZK-4KX."
- note removed: "Cinta 10: GND en 1/3/10. Polarizada. No enchufar con 5 V. 1000uF del modem va en B."
- note removed: "Hay PSU: Q5/Q9 ON -> backup EN=0, Q8 ON, Q10 OFF."
- note removed: "Q3 5V_MODEM. 74HCT125 DIP-14: 1=OE 2=A 3=Y 7=GND 14=VCC. 6/10/13→VCC, 4/9/12→GND."
- note removed: "Sin PSU: Q8 OFF, EN=Gel+, Q11 ON, Q10 ON. Ambos NDP6020P S=BUS D=fuente."
- note removed: "TLC555 HIGH=5V corta Q1. Modem: 74HCT125 DIP (3V3 in, 5V out). Todo THT."
