File: hardware/kicad/01-alimentacion.kicad_sch (KiCad schematic)
At the start: 46 parts, among them J1 PSU 5V 5A, J7 Enlace 5V A, J9 Enlace sig A, Q1 NDP6020P, Q3 NDP6020P, SW1 RESET gabinete, U1 XY-SJVA 6.85V/0.6A, U13 74HCT14, U14 LM66200, U2 XL6019, U3 CD4541BE, U4 TLC555

Commit message: hardware: schematic v1.5.3 nuclear cleanup (water, LEDs, HCT123, layout)
Water on P00 without PC817; IN1/IN2 on both opto channels; LED rails split; HCT_Q separate from TRIG_N; PU/modem spine shorts fixed.

Co-authored-by: Cursor <cursoragent@cursor.com>
Parts:
- removed C17, C4, C5, C8: 100n, symbol Device:C
- removed C6: 10n, symbol Device:C
- removed C7: 100uF, symbol Device:C_Polarized
- removed D10, D3, D4, D5: 1N4148, symbol Device:D
- removed D2: LED GRN PWR, symbol Device:LED
- removed J9: Enlace sig A, symbol Connector_Generic:Conn_01x06
- removed Q3: NDP6020P, symbol Device:Q_PMOS
- removed R11: 22k, symbol Device:R
- removed R12: 10k, symbol Device:R
- removed R20, R24: 100k, symbol Device:R
- removed R5: 330R, symbol Device:R
- removed U13: 74HCT14, symbol Module:HCT14
- removed U3: CD4541BE, symbol Timer:CD4541BE
- removed U4: TLC555, symbol Timer:NE555D
- added C17: 47uF/16V, symbol Device:C_Polarized
- added C18: 2.2uF, symbol Device:C
- added J9: Enlace sig A, symbol Connector_Generic:Conn_01x08
- added Q_DONE, Q_EN: 2N3904, symbol Device:Q_NPN
- added R21: 10k, symbol Device:R
- added R25: 100k, symbol Device:R
- added U3: TPL5010, symbol Module:TPL5010
- added U4: 74HCT123, symbol Module:HCT123
- R10: value 100k -> 10k
- R8: value 1M -> 57.6k
- R9: value 10k -> 100k
Connections:
- net 5V_MODEM is gone; now on net 5V_SYS: J7.4 (Pin_4)
- net MODEM_CUT is gone; now on net IO15: R23.1
- net WDT_MR is gone; now on net 5V_BUS: R10.1
- net WDT_PULSE is gone; now on an unnamed net: R19.1
- net 5V_BUS: now also R10.2, R4.1, Q_DONE.C, R25.1, U3.1 (VDD), U3.3 (DONE), U4.2 (B1), U4.6 (VCC), U4.8 (A2)
- net GEL_ADC: now also J9.1 (Pin_1)
- net GND: now also R8.1, R8.2, C17.2, C18.2, J9.8 (Pin_8), Q_DONE.E, Q_EN.E, U3.2 (GND), U3.6 (DELAY), U4.10 (/CLR2), U4.4 (GND), U4.9 (B2); no longer R10.2, R4.2
- net IO15: now also J9.2 (Pin_2)
- net at R23.2: now also Q_DONE.B
- net at Q1.G, R3.1: no longer R19.2
- net BB_EN: no longer names the net of R2.2, U2.3 (EN)
- net BB_EN: now also Q_EN.C
- net BTN_RESET renamed TRIG_N
- net TRIG_N: now also R9.2, J9.3 (Pin_3), J9.5 (Pin_5), U3.5 (RSTn), U4.1 (A1)
- net PSU_DET: no longer names the net of R1.2, R18.1
- net PSU_DET: now also R21.1
- new net: C18.1, R25.2, U4.3 (/CLR1)
- new net: Q_EN.B, R21.2
- new net: C17.1, R4.2, U4.7 (RCx)
- new net 3V3: J9.6 (Pin_6)
- new net HCT_Q: R19.2, U4.5 (Q)
- new net SPARE: J9.4 (Pin_4)
- new net SPARE2: J9.7 (Pin_7)
- no-connect marks 6 -> 2
Other:
- note added: "A1=TRIG_N (PU 100k). Q=HCT_Q→R19→Q1. RCx=100k+47u ~2s. /CLR blank 100k+2.2u."
- note added: "Ajuste XL6019 5,1 V. No XL6009 / ZK-4KX. Sin HCT14 / D10."
- note added: "Bloques: carga | backup+OR | Q1+74HCT123 | TPL5010@5V_BUS. Labels entre bloques."
- note added: "CallOnFail v1.5.3 — alimentacion (proto)"
- note added: "DONE OD: IO15 alto→DONE bajo; pateo IO15 bajo. REXT 57.6k≈10 min. /CLR blank 100k+2.2u."
- note added: "J9: GEL_ADC IO15 TRIG_N SPARE TRIG_N 3V3 SPARE2 GND."
- note added: "Nuclear: TRIG_N→A1 (flanco↓) · Q→HCT_Q→1k→Q1 (~2s OFF). A1≠Q."
- note added: "OR: LM66200 (VIN1=PSU, VIN2=XL6019). R2=pull-up Gel+→EN; Q_EN hunde EN→GND si hay PSU."
- note added: "Proto A↔B: J7 bornera 5,08 (GND 5V_SYS GND 5V_SYS) + J9 Molex. Modem=SYS."
- note added: "Q1 idle ON. SW1→TRIG_N. LED PWR en hoja I/O."
- note added: "TPL5010 @5V_BUS ~10 min. DONE←NPN←IO15. RSTn→TRIG_N."
- note removed: "Ajuste XL6019 5,1 V. No XL6009 / ZK-4KX. Modulo AE con pines 2,54."
- note removed: "Bloques: carga | backup | high-side | WDT. Cable corto dentro del bloque; global al cruzar hoja."
- note removed: "CallOnFail v1 — alimentacion (proto)"
- note removed: "D5: timeout 4541 baja TRIG. SW1 NA a GND. TLC555 OUT a Q1 (no NE555 bipolar)."
- note removed: "LED PWR de frente, sin ESP."
- note removed: "No cinta IDC. No 5V_BUS / 3V3 / GEL+. Luego una placa: estas nets son pistas."
- note removed: "OR: LM66200 (VIN1=PSU, VIN2=XL6019). EN=0 con PSU (HCT14+D10). R2 a Gel+."
- note removed: "Patada IO15 acople. No DC a GND en IO15. R20 baja MR."
- note removed: "Proto A↔B: J7 bornera 5,08 (GND 5V_SYS GND 5V_MODEM) + J9 Molex KK 2,54 o bornera."
- note removed: "Q1 5V_SYS. 555 idle LOW = ON. Pulso HIGH ~2 s = OFF."
- note removed: "Q3 5V_MODEM. HCT14: 2Y->3A = buffer. D10: 1Y baja BB_EN (R2 a Gel+)."
- note removed: "R8/C4: tunear 4-5 min (2^16). Pin 9 HIGH => Q activo bajo. C8 junto al 4541."
- note removed: "TLC555->Q1. 74HCT14: 1=EN backup, 2+3=buffer MODEM_CUT. Solo 2x NDP6020P."
- note removed: "WDT CD4541 (~4-5 min) + TLC555 CMOS (~2 s) en 5V_BUS"
- title: CallOnFail v1 — Alimentacion -> CallOnFail v1.5.3 — Alimentacion
