File: hardware/kicad/01-alimentacion.kicad_sch (KiCad schematic)
At the start: 34 parts, among them J1 PSU 5V 5A, J7 Enlace 5V A, J9 Enlace sig A, Q1 NDP6020P, SW1 RESET gabinete, U1 XY-SJVA 6.85V/0.6A, U14 LM66200, U2 XL6019, U3 TPL5010, U4 74HCT123

Commit message: hardware: sync KiCad schematics after manual edits
Hand-tuned hierarchical sheets and project settings; source of truth for v1.5 layout.

Co-authored-by: Cursor <cursoragent@cursor.com>
Connections:
- net 5V_BUS: no longer Q_DONE.C, R10.2, U3.3 (DONE)
- net GEL_P: no longer F1.2, R6.1
- net GND: now also R3.1; no longer R3.2, R8.1, U3.6 (DELAY)
- net at Q1.G, R19.1: now also R3.2; no longer R3.1
- new net: F1.2, R6.1
- new net: R8.1, U3.6 (DELAY)
- new net: Q_DONE.C, R10.2, U3.3 (DONE)
Other:
- moved on the sheet: BT1, C1, C10, C17, C18, C3, C9, F1, J1, J7, J9, Q1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
