File: hardware/kicad/02-io.kicad_sch (KiCad schematic)
At the start: 25 parts, among them J2 USB-Serial 3V3, J3 MODEM_CUT GPIO, J4 Campo IN/OUT, J5 Campo GND/COM, J6 Panel 5 pin, K1 OUT1 sirena, K2 OUT2 aux, SW2 Servicio IO39, U10 ZMPT101B, U11 PCF8574, U12 ULN2003, U5 WT32-ETH01, U6 A7672SA-FASE, U7 OLED 0x3C, U8 SHT31 0x44, U9 DS18B20 x4

Commit message: Lock v1 proto hardware: 5 V MOSFET OR, THT parts, 2 IN / 2 OUT, independent buzzer.
PCF keeps NET and ALARM LEDs; buzzer is P3 via ULN so a rule can sound without closing field relays.

Co-authored-by: Cursor <cursoragent@cursor.com>
Parts:
- removed J4: Campo IN/OUT, symbol Connector_Generic:Conn_01x06
- added C11, C12, C13, C14: 100n, symbol Device:C
- added C15: 10uF, symbol Device:C_Polarized
- added C2: 1000uF/16V, symbol Device:C_Polarized
- added J4: Campo IN/OUT, symbol Connector_Generic:Conn_01x04
- added J8: IDC B←A, symbol Module:IDC10
- added LS1: Buzzer 5V activo, symbol Module:BUZZER
- added R27, R28, R29, R31: 10k, symbol Device:R
- added R32, R33, R34: 1k, symbol Device:R
- K1: value OUT1 sirena -> OUT1
Connections:
- net 3V3: now also C13.1, R27.1, R28.1, R29.1, R31.1
- net 5V_MODEM: now also C12.1, C2.1, J8.4 (5V_MODEM)
- net 5V_SYS: now also C11.1, C15.1, J8.2 (5V_SYS), LS1.1 (+); no longer D6.2 (A), D7.2 (A), J6.3 (Pin_3), J6.4 (Pin_4), R16.2, R17.2
- net BTN_RESET: now also J8.9 (BTN_RESET)
- net BTN_SVC: now also R31.2
- net GEL_ADC: now also J8.5 (GEL_ADC)
- net GND: now also C11.2, C12.2, C13.2, C14.2, C15.2, C2.2, J8.1 (GND), J8.10 (GND), J8.3 (GND); no longer U12.3 (I3)
- net IO15: now also J8.6 (IO15)
- net LED_ALM: now also J6.4 (Pin_4)
- net LED_NET: now also J6.3 (Pin_3)
- net LED_PWR: now also J8.8 (LED_PWR)
- net MODEM_CUT: now also J8.7 (MODEM_CUT)
- net ZMPT_ADC: now also C14.1, R34.2; no longer U10.1 (OUT)
- net at J5.2 (Pin_2), K1.3 (COM), K1.4 (NO)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: now also J4.3 (Pin_3), J4.4 (Pin_4); no longer U11.10 (P2), U11.11 (P3), U11.8 (P0), U11.9 (P1)
- net at U12.14 (O3): now also LS1.2 (-)
- net at U5.7 (IO2), U5.8 (IO4), U6.5 (RESET)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: now also R32.1, R32.2, R33.1, R33.2; no longer U5.12 (IO17), U5.9 (IO5), U6.3 (TXD), U6.4 (RXD)
- new net: J4.1 (Pin_1), J4.2 (Pin_2), R27.2, R28.2, U11.8 (P0), U11.9 (P1)
- new net: D6.2 (A), R16.2
- new net: D7.2 (A), R17.2
- new net: R29.2, U11.10 (P2)
- new net: R34.1, U10.1 (OUT)
- new net: U5.12 (IO17), U6.4 (RXD)
- new net: U5.9 (IO5), U6.3 (TXD)
- new net BUZZ_DRV: U11.11 (P3), U12.3 (I3)
- no-connect marks 7 -> 6
Other:
- note added: "IN1 fuga, IN2 extra. P2 spare 10k. Contacto seco a GND."
- note added: "IO39 sin pull interno. 10k a 3V3. Corta=llamada, larga=OTA."
- note added: "J2: USB TX->RXD0, USB RX->TXD0, IO0 a GND solo para flash. No 5V del USB."
- note added: "J3: GPIO salida TBD (no IO39, no IO2, no strapping). HIGH = corta modem."
- note added: "OC IO4/IO2 via 1k. No >100 nF. No bajar RESET y PWRKEY a la vez."
- note added: "P3=buzzer O3, P4=K1 O1, P5=K2 O2. P6=NET P7=ALARMA. 2 IN + 2 OUT."
- note added: "Panel: GND, PWR, NET (P6), ALARMA (P7), RESET. Buzzer P3, no borne."
- note added: "ZMPT OUT -> 1k -> IO36. No 220 hasta validar."
- note removed: "Corta=llamada, larga=OTA."
- note removed: "IN1 fuga. Contacto seco a GND."
- note removed: "J2: USB TX->RXD0, USB RX->TXD0, IO0 a GND solo para flash."
- note removed: "J3: GPIO de salida TBD (no IO39, no IO2)."
- note removed: "OC IO4/IO2. No >100 nF. No bajar RESET y PWRKEY a la vez."
- note removed: "Panel: GND, PWR, NET (P6), ALARMA (P7), RESET."
- note removed: "ULN sink + 1N4007. COM ULN a 5V_SYS."
- note removed: "ZMPT OUT -> IO36."

Commit message: Stop tracking PDFs and generated KiCad dumps; set WiFi from the web over Ethernet.
Vendor manuals, schematic PDFs, SVG previews and ERC reports do not belong in git or agent context. Firmware prefers Ethernet and accepts set_wifi/clear_wifi from the device page.

Co-authored-by: Cursor <cursoragent@cursor.com>
Parts:
- removed J8: IDC B←A, symbol Module:IDC10
- added J10: Enlace sig B, symbol Connector_Generic:Conn_01x06
- added J8: Enlace 5V B, symbol Connector_Generic:Conn_01x04
Connections:
- net 5V_MODEM: now also J8.4 (Pin_4)
- net 5V_SYS: now also J8.2 (Pin_2)
- net BTN_RESET: now also J10.5 (Pin_5)
- net GEL_ADC: now also J10.1 (Pin_1)
- net GND: now also J10.6 (Pin_6), J8.1 (Pin_1), J8.3 (Pin_3)
- net IO15: now also J10.2 (Pin_2)
- net LED_PWR: now also J10.4 (Pin_4)
- net MODEM_CUT: now also J10.3 (Pin_3)
- net at R32.1, R32.2, R33.2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: no longer R33.1, U5.7 (IO2)
- net I2C_SDA: now reaches R13.2, U11.3 (SDA), U5.13 (IO32), U7.3 (SDA), U8.3 (SDA)
- net I2C_SCL: now reaches R14.2, U11.4 (SCL), U5.14 (IO33), U7.4 (SCL), U8.4 (SCL)
- net UART_TX: now reaches U5.12 (IO17), U6.4 (RXD)
- net UART_RX: now reaches U5.9 (IO5), U6.3 (TXD)
- new net: R33.1, U5.7 (IO2)
Other:
- note added: "Mismo pinout que J7/J9. Cable 0,75 mm2 en 5 V. Molex polarizado o bornera, no IDC."
