File: hardware/kicad/02-io.kicad_sch (KiCad schematic)
At the start: 41 parts, among them J10 Enlace sig B, J2 USB-Serial 3V3, J3 MODEM_CUT GPIO, J4 Campo IN/OUT, J5 Campo GND/COM, J6 Panel 5 pin, J8 Enlace 5V B, K1 OUT1, K2 OUT2 aux, SW2 Servicio IO39, U10 ZMPT101B, U11 PCF8574, U12 ULN2003, U5 WT32-ETH01, U6 A7672SA-FASE, U7 OLED 0x3C, U8 SHT31 0x44, U9 DS18B20 x4

Commit message: hardware: schematic v1.5.3 nuclear cleanup (water, LEDs, HCT123, layout)
Water on P00 without PC817; IN1/IN2 on both opto channels; LED rails split; HCT_Q separate from TRIG_N; PU/modem spine shorts fixed.

Co-authored-by: Cursor <cursoragent@cursor.com>
Parts:
- removed D9: 1N4007, symbol Device:D
- removed J10: Enlace sig B, symbol Connector_Generic:Conn_01x06
- removed J2: USB-Serial 3V3, symbol Connector_Generic:Conn_01x04
- removed J4: Campo IN/OUT, symbol Connector_Generic:Conn_01x04
- removed J5: Campo GND/COM, symbol Connector_Generic:Conn_01x02
- removed J6: Panel 5 pin, symbol Connector_Generic:Conn_01x05
- removed K1: OUT1, symbol Module:RELAY
- removed K2: OUT2 aux, symbol Module:RELAY
- removed R31: 10k, symbol Device:R
- removed U11: PCF8574, symbol Module:PCF8574
- removed U12: ULN2003, symbol Transistor_Array:ULN2003
- added D2: LED GRN PWR, symbol Device:LED
- added D9: LED LTE, symbol Device:LED
- added J10: Enlace sig B, symbol Connector_Generic:Conn_01x08
- added J11: RS485 A/B, symbol Connector_Generic:Conn_01x02
- added J4: Campo IN2, symbol Connector_Generic:Conn_01x02
- added J5: Campo OUT, symbol Connector_Generic:Conn_01x04
- added J6: Panel 6 pin, symbol Connector_Generic:Conn_01x06
- added K1: 2-relay opto, symbol Module:RELAY2_OPTO
- added Q_BZ: 2N3904, symbol Device:Q_NPN
- added R26, R5: 330R, symbol Device:R
- added R30: 10k, symbol Device:R
- added R35: 15k, symbol Device:R
- added R36: 1k, symbol Device:R
- added SW_BOOT: BOOT IO0, symbol Switch:SW_Push
- added SW_EN: EN reset, symbol Switch:SW_Push
- added U11: PCF8575, symbol Module:PCF8575
- added U12: PC817 2CH, symbol Module:PC817_2CH
- added U15: FT232, symbol Module:FT232
- added U16: RS485 auto, symbol Module:RS485
- added U17: Water det, symbol Module:WATER_DET
- D8: value 1N4007 -> 1N4148
- J3: value MODEM_CUT GPIO -> Campo IN1
- R34: value 1k -> 10k
- SW2: value Servicio IO39 -> Servicio P02
Connections:
- net 5V_MODEM is gone; now on net 5V_SYS: C12.1, C2.1, J8.4 (Pin_4), U6.1 (VCC)
- net 3V3: now also R16.1, R17.1, R27.2, R28.2, R29.2, J10.6 (Pin_6), K1.1 (VCC), R26.1, R30.2, U11.1 (VCC), U12.6 (VCC), U16.1 (VCC); no longer R27.1, R28.1, R29.1
- net 5V_SYS: now also U10.1 (VCC), K1.2 (JD-VCC), R5.1, U17.1 (VCC); no longer D8.1 (K), R16.1, R17.1
- net GEL_ADC: now also U5.17 (IO35), J10.1 (Pin_1); no longer U5.15 (IO35)
- net GND: now also D2.1 (K), J10.8 (Pin_8), J6.1 (Pin_1), K1.3 (GND), Q_BZ.E, R35.2, SW_BOOT.2, SW_EN.2, U11.2 (GND), U11.5 (A0), U11.6 (A1), U11.7 (A2), U12.7 (GND), U15.1 (GND), U16.2 (GND), U17.2 (GND), U17.5 (COM); no longer J3.2 (Pin_2)
- net I2C_SCL: now also U5.16 (IO33), U11.4 (SCL); no longer U5.14 (IO33)
- net I2C_SDA: now also U5.15 (IO32), U11.3 (SDA); no longer U5.13 (IO32)
- net IO15: now also U5.13 (IO15), J10.2 (Pin_2); no longer U5.11 (IO15)
- net LED_PWR: now also D2.2 (A), J6.2 (Pin_2), R5.2
- net at LS1.2 (-): now also Q_BZ.C
- net PHY_NRST: now reaches D8.2 (A)
- net at R34.1: now also U10.3 (OUT); no longer U10.1 (OUT)
- net at R33.1: now also U5.8 (IO2); no longer U5.7 (IO2)
- net BTN_SVC renamed PCF_P02
- net PCF_P02: now also R29.1, U11.10 (P02); no longer U5.17 (IO39)
- net LED_ALM renamed PCF_P07
- net PCF_P07: now also J6.4 (Pin_4), U11.15 (P07)
- net LED_NET renamed PCF_P06
- net PCF_P06: now also J6.3 (Pin_3), U11.14 (P06)
- net MODEM_CUT renamed IN1
- net IN1: now also U12.1 (IN1)
- net OWIRE renamed OW_DATA
- net OW_DATA: now also U5.12 (IO14); no longer U5.10 (IO14)
- net UART_RX: no longer names the net of U5.9 (IO4)
- net UART_RX: now also R32.1; no longer U6.3 (TXD)
- net UART_TX renamed MODEM_TX
- net MODEM_TX: now also U5.14 (IO17); no longer U5.12 (IO17)
- net ZMPT_ADC renamed IO36
- net IO36: now also U5.18 (IO36), R35.1; no longer U5.16 (IO36)
- new net: Q_BZ.B, R36.2
- new net: J11.1 (Pin_1), U16.5 (A)
- new net: J11.2 (Pin_2), U16.6 (B)
- new net: D8.1 (K), U11.17 (P11)
- new net: U15.3 (RXD), U5.4 (TXD0)
- new net: U15.2 (TXD), U5.5 (RXD0)
- new net: D9.2 (A), R26.2
- new net EN_SW: SW_EN.1, U5.7 (EN)
- new net FIELD_COM1: J5.1 (Pin_1), K1.6 (COM1)
- new net FIELD_COM2: J5.3 (Pin_3), K1.8 (COM2)
- new net IN2: J4.1 (Pin_1), U12.2 (IN2)
- new net IO0_BOOT: SW_BOOT.1, U5.6 (IO0)
- new net MODEM_PWRKEY: R33.2, U6.6 (PWRKEY)
- new net MODEM_RST: R32.2, U6.5 (RESET)
- new net MODEM_RX: U5.10 (IO5), U6.3 (TXD)
- new net OPTO_COM: J3.2 (Pin_2), J4.2 (Pin_2), U12.3 (GND_F)
- new net OUT1: J5.2 (Pin_2), K1.7 (NO1)
- new net OUT2: J5.4 (Pin_4), K1.9 (NO2)
- new net PCF_P00: R27.1, U11.8 (P00), U17.4 (NO)
- new net PCF_P01: R28.1, U11.9 (P01), U12.4 (OUT1)
- new net PCF_P03: R36.1, U11.11 (P03)
- new net PCF_P04: K1.4 (IN1), U11.12 (P04)
- new net PCF_P05: K1.5 (IN2), U11.13 (P05)
- new net PCF_P10: D9.1 (K), J6.5 (Pin_5), U11.16 (P10)
- new net PCF_P13: R30.1, U11.19 (P13), U12.5 (OUT2)
- new net RS485_RX: U16.4 (RXD), U5.19 (IO39)
- new net RS485_TX: U16.3 (TXD), U5.11 (IO12)
- new net SPARE: J10.4 (Pin_4)
- new net SPARE2: J10.7 (Pin_7)
- new net TRIG_N: J10.3 (Pin_3), J10.5 (Pin_5), J6.6 (Pin_6), U11.18 (P12)
- no-connect marks 6 -> 8
Other:
- note added: "CallOnFail v1.5.3 — WT32, FT232, A7672, PCF8575, campo"
- note added: "ETH_RST: 1N4148→PHY nRST (R43). P12→TRIG_N."
- note added: "FT232 rot180: TXD→RXD0, RXD←TXD0 (cables cortos). No 5V USB. EN=lab."
- note added: "FT232/BOOT/EN | WT32 | modem — I2C/sensores — PCF / campo / panel / RS485."
- note added: "GPIO: 0 BOOT 2 PWRKEY 4 RESET 5/17 modem 12/39 RS485 14 1-Wire 15 DONE 32/33 I2C 35 gel 36 ZMPT EN=lab P12=TRIG_N↓"
- note added: "I2C IO32/IO33. PCF8575 VCC=3V3 dir 0x20. A0-A2 GND."
- note added: "IO15→J10.2→Q_DONE. P12/BTN→TRIG_N. Labels entre bloques (no cables largos)."
- note added: "IO4/IO2 via 1k. Modem VCC=5V_SYS (nuclear Q1). UART/RST=labels."
- note added: "P14-P17 NC. P13=IN2 (opto)."
- note added: "Panel: PWR=5V_SYS→330→LED→GND (J6.2=LED_PWR). NET/ALARM/LTE=3V3→330→LED→PCF (J6=cátodo). Sin mezclar rieles."
- note added: "RS485: IO12 TX, IO39 RX (labels). Servicio = PCF P02."
- note added: "Servicio P02: input lab/mantenimiento. No RESET. No silencia alarmas."
- note added: "Water→P00 directo. PC817=IN1→P01 + IN2→P13. Buzzer P03→NPN."
- note added: "ZMPT OUT→10k→IO36; 15k+100n GND. No 220 hasta validar."
- note added: "jumper VCC-JD-VCC OFF"
- note removed: "CallOnFail v1 — WT32, A7672, sensores, PCF, frente"
- note removed: "GPIO: 0 ETH CLK 2 PWRKEY 4 RESET 5 RX 14 1-Wire 15 WDT 16/18/23 ETH 17 TX 32 SDA 33 SCL 35 gel 36 ZMPT 39 servicio"
- note removed: "I2C IO32/IO33. Pull-up 4k7; omitir si el modulo ya las trae. PCF 0x20."
- note removed: "IN1 fuga, IN2 extra. P2 spare 10k. Contacto seco a GND."
- note removed: "IO39 sin pull interno. 10k a 3V3. Corta=llamada, larga=OTA."
- note removed: "J2: USB TX->RXD0, USB RX->TXD0, IO0 a GND solo para flash. No 5V del USB."
- note removed: "J3: GPIO salida TBD (no IO39, no IO2, no strapping). HIGH = corta modem."
- note removed: "OC IO4/IO2 via 1k. No >100 nF. No bajar RESET y PWRKEY a la vez."
- note removed: "P3=buzzer O3, P4=K1 O1, P5=K2 O2. P6=NET P7=ALARMA. 2 IN + 2 OUT."
- note removed: "Panel: GND, PWR, NET (P6), ALARMA (P7), RESET. Buzzer P3, no borne."
- note removed: "USB | WT32 | modem — I2C y sensores debajo — PCF / campo / relés a la derecha."
- note removed: "ZMPT OUT -> 1k -> IO36. No 220 hasta validar."
- title: CallOnFail v1 — ESP32 / modem / sensores / campo -> CallOnFail v1.5.3 — ESP32 / modem / sensores / campo
