File: hardware/kicad/02-io.kicad_sch (KiCad schematic)
At the start: 51 parts, among them J10 Enlace sig B, J11 RS485 A/B, J3 Campo IN1, J4 Campo IN2, J5 Campo OUT, J6 Panel 6 pin, J8 Enlace 5V B, K1 2-relay opto, SW2 Servicio P02, U10 ZMPT101B, U11 PCF8575, U12 PC817 2CH, U15 FT232, U16 RS485 auto, U17 Water det, U5 WT32-ETH01, U6 A7672SA-FASE, U7 OLED 0x3C, U8 SHT31 0x44, U9 DS18B20 x4

Commit message: hardware: sync KiCad schematics after manual edits
Hand-tuned hierarchical sheets and project settings; source of truth for v1.5 layout.

Co-authored-by: Cursor <cursoragent@cursor.com>
Connections:
- net 5V_SYS: no longer R5.1
Other:
- note removed: "CallOnFail v1.5.3 — WT32, FT232, A7672, PCF8575, campo"
- note removed: "FT232/BOOT/EN | WT32 | modem — I2C/sensores — PCF / campo / panel / RS485."
- note removed: "IO15→J10.2→Q_DONE. P12/BTN→TRIG_N. Labels entre bloques (no cables largos)."
- moved on the sheet: C11, C12, C13, C14, C15, C2, D2, D6, D7, D8, D9, J11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
