File: hardware/kicad/cof-v1.kicad_sch (KiCad schematic)
At the start: 0 parts

Commit message: hardware: schematic v1.5.3 nuclear cleanup (water, LEDs, HCT123, layout)
Water on P00 without PC817; IN1/IN2 on both opto channels; LED rails split; HCT_Q separate from TRIG_N; PU/modem spine shorts fixed.

Co-authored-by: Cursor <cursoragent@cursor.com>
Other:
- note added: "5V_PSU 5V_BUS 5V_SYS 3V3 GEL_P GEL_ADC IO15 TRIG_N HCT_Q PHY_NRST"
- note added: "CallOnFail hardware v1.5.3"
- note added: "Dos hojas: A alimentacion+TPL+123 + B I/O. Enlace proto bornera/Molex. Luego una placa."
- note added: "Rev 1.5.3: sin Q3; modem=SYS; TPL@BUS+NPN; 74HCT123~2s→Q1; P12 SYS_KILL↓; EN=lab."
- note removed: "5V_PSU 5V_BUS 5V_SYS 5V_MODEM 3V3 GEL_P GEL_ADC IO15 MODEM_CUT LED_PWR BTN_RESET"
- note removed: "CallOnFail hardware v1"
- note removed: "Dos hojas: A alimentacion + B I/O. Enlace proto bornera/Molex. Luego una placa."
- note removed: "No 12 V. No ZK-S4. No XL4015. No IRF4905 a 5 V. Gel 6 V 7 Ah, flote 6,85 V."
- title: CallOnFail v1 -> CallOnFail v1.5.3
Changed lines of the file:
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@@
 	(paper "A3")
 	(title_block
-		(title "CallOnFail v1")
-		(date "2026-09-12")
-		(rev "1.4")
+		(title "CallOnFail v1.5.3")
+		(date "2026-10-04")
+		(rev "1.5.3")
 		(company "CallOnFail")
-		(comment 1 "WT32-ETH01 + A7672SA-FASE + gel 6V. Ver docs/HARDWARE_V1.md")
+		(comment 1 "WT32 + A7672 + gel 6V + TPL5010 + 74HCT123 + PCF8575. Ver docs/HARDWARE_V1.md")
 	)
-	(text "5V_PSU  5V_BUS  5V_SYS  5V_MODEM  3V3  GEL_P  GEL_ADC  IO15  MODEM_CUT  LED_PWR  BTN_RESET"
+	(text "CallOnFail hardware v1.5.3"
 		(exclude_from_sim no)
-		(at 50.8 48.26 0)
-		(effects
-			(font
-				(size 1.27 1.27)
-			)
-			(justify left bottom)
-		)
+		(at 50.80 30.48 0)
+		(effects (font (size 3.81 3.81)) (justify left bottom))
 	)
-	(text "CallOnFail hardware v1"
+	(text "Dos hojas: A alimentacion+TPL+123 + B I/O. Enlace proto bornera/Molex. Luego una placa."
 		(exclude_from_sim no)
-		(at 50.8 30.48 0)
-		(effects
-			(font
-				(size 3.81 3.81)
-			)
-			(justify left bottom)
-		)
+		(at 50.80 40.64 0)
+		(effects (font (size 1.27 1.27)) (justify left bottom))
 	)
-	(text "No 12 V. No ZK-S4. No XL4015. No IRF4905 a 5 V. Gel 6 V 7 Ah, flote 6,85 V."
+	(text "5V_PSU  5V_BUS  5V_SYS  3V3  GEL_P  GEL_ADC  IO15  TRIG_N  HCT_Q  PHY_NRST"
 		(exclude_from_sim no)
-		(at 50.8 55.88 0)
-		(effects
-			(font
-				(size 1.27 1.27)
-			)
-			(justify left bottom)
-		)
+		(at 50.80 48.26 0)
+		(effects (font (size 1.27 1.27)) (justify left bottom))
 	)
-	(text "Dos hojas: A alimentacion + B I/O. Enlace proto bornera/Molex. Luego una placa."
+	(text "Rev 1.5.3: sin Q3; modem=SYS; TPL@BUS+NPN; 74HCT123~2s→Q1; P12 SYS_KILL↓; EN=lab."
 		(exclude_from_sim no)
-		(at 50.8 40.64 0)
-		(effects
-			(font
-				(size 1.27 1.27)
-			)
-			(justify left bottom)
-		)
+		(at 50.80 55.88 0)
+		(effects (font (size 1.27 1.27)) (justify left bottom))
 	)
 	(sheet
-		(at 50.8 76.2)
+		(at 50.80 76.20)
 		(size 71.12 40.64)
 		(exclude_from_sim no)
@@
 		(on_board yes)
 		(dnp no)
-		(stroke
-			(width 0.1524)
-			(type solid)
-		)
-		(fill
-			(color 0 0 0 0)
-		)
+		(stroke (width 0.1524) (type solid))
+		(fill (color 0 0 0 0.0000))
 		(property "Sheetname" "Alimentacion"
-			(at 50.8 75 0)
-			(show_name no)
-			(do_not_autoplace no)
-			(effects
-				(font
-					(size 1.27 1.27)
-				)
-				(justify left bottom)
-			)
+			(at 50.80 75.00 0)
+			(effects (font (size 1.27 1.27)) (justify left bottom))
 		)
 		(property "Sheetfile" "01-alimentacion.kicad_sch"
-			(at 50.8 117.5 0)
-			(show_name no)
-			(do_not_autoplace no)
-			(effects
-				(font
-					(size 1.27 1.27)
-				)
-				(justify left top)
-			)
+			(at 50.80 117.50 0)
+			(effects (font (size 1.27 1.27)) (justify left top))
 		)
 	)
 	(sheet
-		(at 160.02 76.2)
+		(at 160.02 76.20)
 		(size 81.28 40.64)
 		(exclude_from_sim no)
@@
 		(on_board yes)
 		(dnp no)
-		(stroke
-			(width 0.1524)
-			(type solid)
-		)
-		(fill
-			(color 0 0 0 0)
-		)
+		(stroke (width 0.1524) (type solid))
+		(fill (color 0 0 0 0.0000))
 		(property "Sheetname" "ESP32 modem sensores"
-			(at 160.02 75 0)
-			(show_name no)
-			(do_not_autoplace no)
-			(effects
-				(font
-					(size 1.27 1.27)
-				)
-				(justify left bottom)
-			)
+			(at 160.02 75.00 0)
+			(effects (font (size 1.27 1.27)) (justify left bottom))
 		)
 		(property "Sheetfile" "02-io.kicad_sch"
-			(at 160.02 117.5 0)
-			(show_name no)
-			(do_not_autoplace no)
-			(effects
-				(font
-					(size 1.27 1.27)
-				)
-				(justify left top)
-			)
+			(at 160.02 117.50 0)
+			(effects (font (size 1.27 1.27)) (justify left top))
 		)
 	)
@@
 		)
 	)
+	(embedded_fonts no)
 )
